Commit message: update bongo board

File: gym/envs/dart/assets/darwinmodel/bongo_board.urdf (robot description, URDF)
Before this commit: robot bongo_board_skeleton, 3 links, 2 joints
Links:
- link board: mass 0.5 -> 0.453; geometry collision box size=0.15 0.4 0.01; visual box size=0.15 0.4 0.01
- link support: mass 0.25 -> 0.151; geometry collision cylinder length=0.15 radius=0.035; visual cylinder length=0.15 radius=0.035
Joints:
- joint jt1: origin xyz=0 0 -0.28 rpy=0 0 0 -> xyz=0 0 -0.27 rpy=0 0 0

File: gym/envs/dart/assets/darwinmodel/ground1.urdf (robot description, URDF)
Before this commit: robot ground_skeleton, 6 links, 5 joints
Links:
- removed link pillar1
- removed link pillar2
- removed link pillar3
- added link wall, mass 1.0; collision box size=125 25 0.1; visual box size=125 25 0.1
Joints:
- removed joint pillar1joint
- removed joint pillar2joint
- removed joint pillar3joint
- added joint ground_joint_wall: type fixed, parent ground_link, child wall, origin xyz=0 0 0 rpy=0 0 0

File: gym/envs/dart/assets/darwinmodel/tracking_box.urdf (robot description, URDF)
Before this commit: robot track_box_skeleton, 4 links, 3 joints
Links:
- link track_box: geometry 

Commit message: update a bit

File: gym/envs/dart/assets/darwinmodel/bongo_board.urdf (robot description, URDF)
Before this commit: robot bongo_board_skeleton, 3 links, 2 joints
Links:
- link support: geometry collision cylinder length=0.15 radius=0.015; visual cylinder length=0.15 radius=0.015
Joints:
- joint jt1: origin xyz=0 0 -0.27 rpy=0 0 0 -> xyz=0 0 -0.31 rpy=0 0 0

File: gym/envs/dart/assets/darwinmodel/ground1.urdf (robot description, URDF)
Before this commit: robot ground_skeleton, 4 links, 3 joints
Links:
- added link pillar1, mass 1.0; visual box size=0.1 0.1 10.0
- added link pillar2, mass 1.0; visual box size=0.1 0.1 10.0
- added link pillar3, mass 1.0; visual box size=0.1 0.1 10.0
- link wall: geometry visual box size=125 25 0.1
Joints:
- added joint pillar1joint: type fixed, parent ground_link, child pillar1, origin xyz=0 0 0 rpy=0 0 0
- added joint pillar2joint: type fixed, parent ground_link, child pillar2, origin xyz=0 0 0 rpy=0 0 0
- added joint pillar3joint: type fixed, parent ground_link, child pillar3, origin xyz=0 0 0 rpy=0 0 0

Commit message: add soft ground to darwin

File: gym/envs/dart/assets/darwinmodel/bongo_board.urdf (robot description, URDF)
Before this commit: robot bongo_board_skeleton, 3 links, 2 joints
Links:
- link support: geometry collision cylinder length=0.15 radius=0.035; visual cylinder length=0.15 radius=0.035
Joints:
- joint jt1: origin xyz=0 0 -0.31 rpy=0 0 0 -> xyz=0 0 -0.27 rpy=0 0 0
