Commit message: add soft ground and movable ground

File: gym/envs/dart/assets/darwinmodel/soft_ground.urdf (robot description, URDF)
Before this commit: robot ground_skeleton, 2 links, 1 joints
Links:
- link ground_link: geometry visual box size=125 25 2.05

File: gym/envs/dart/assets/robotis_op3/robotis_op3.urdf (robot description, URDF)
Before this commit: robot robotis_op3, 23 links, 22 joints
Links:
- link body_link: geometry collision box size=0.1745 0.1288 0.14529999; visual mesh filename=./meshes/body_simp.stl scale=0.001 0.001 0.001
- link head_pan_link: geometry collision box size=0.0325 0.042 0.031; visual mesh filename=./meshes/h1_simp.stl scale=0.001 0.001 0.001
- link head_tilt_link: geometry collision box size=0.0445 0.094 0.078; visual mesh filename=./meshes/h2_simp.stl scale=0.001 0.001 0.001
- link l_ank_pitch_link: geometry collision box size=0.079 0.0424 0.0465; visual mesh filename=./meshes/ll5_simp.stl scale=0.001 0.001 0.001
- link l_ank_roll_link: geometry collision box size=0.127 0.08 0.01; visual mesh filename=./meshes/ll6_simp.stl scale=0.001 0.001 0.001
- link l_el_link: geometry collision box size=0.042 0.14900986 0.03; visual mesh filename=./meshes/la3_simp.stl scale=0.001 0.001 0.001
- link l_hip_pitch_link: geometry collision box size=0.03085 0.0464 0.1239; visual mesh filename=./meshes/ll3_simp.stl scale=0.001 0.001 0.001
- link l_hip_roll_link: geometry collision box size=0.07975 0.0424 0.0465; visual mesh filename=./meshes/ll2_simp.stl scale=0.001 0.001 0.001
- link l_hip_yaw_link: geometry collision box size=0.045 0.025 0.031; visual mesh filename=./meshes/ll1_simp.stl scale=0.001 0.001 0.001
- link l_knee_link: geometry collision box size=0.03 0.044 0.115; visual mesh filename=./meshes/ll4_simp.stl scale=0.001 0.001 0.001
- link l_sho_pitch_link: geometry collision box size=0.042 0.031 0.0325; visual mesh filename=./meshes/la1_simp.stl scale=0.001 0.001 0.001
- link l_sho_roll_link: geometry collision box size=0.0424 0.1129 0.0301; visual mesh filename=./meshes/la2_simp.stl scale=0.001 0.001 0.001
- link r_ank_pitch_link: geometry collision box size=0.07975 0.0424 0.0465; visual mesh filename=./meshes/rl5_simp.stl scale=0.001 0.001 0.001
- link r_ank_roll_link: geometry collision box size=0.127 0.08 0.01; visual mesh filename=./meshes/rl6_simp.stl scale=0.001 0.001 0.001
- link r_el_link: geometry collision box size=0.042 0.14900986 0.03; visual mesh filename=./meshes/ra3_simp.stl scale=0.001 0.001 0.001
- link r_hip_pitch_link: geometry collision box size=0.03085 0.0464 0.1239; visual mesh filename=./meshes/rl3_simp.stl scale=0.001 0.001 0.001
- link r_hip_roll_link: geometry collision box size=0.07975 0.0424 0.0465; visual mesh filename=./meshes/rl2_simp.stl scale=0.001 0.001 0.001
- link r_hip_yaw_link: geometry collision box size=0.045 0.025 0.031; visual mesh filename=./meshes/rl1_simp.stl scale=0.001 0.001 0.001
- link r_knee_link: geometry collision box size=0.03 0.044 0.115; visual mesh filename=./meshes/rl4_simp.stl scale=0.001 0.001 0.001
- link r_sho_pitch_link: geometry collision box size=0.042 0.031 0.0325; visual mesh filename=./meshes/ra1_simp.stl scale=0.001 0.001 0.001
- link r_sho_roll_link: geometry collision box size=0.0424 0.1129 0.0301; visual mesh filename=./meshes/ra2_simp.stl scale=0.001 0.001 0.001
